File: KiCAD/RESTfan/RESTfan.kicad_pcb (KiCad board)
At the start: 2 copper layers, 75 x 81.5 mm, 22 parts, among them J1 Conn_01x02_Male, J2 Conn_01x03_Male, J3 Conn_01x03_Male, K1 FINDER-30.22, K2 FINDER-30.22, K3 FINDER-30.22, K4 FINDER-30.22, Q1 BSS138, Q2 BSS138, Q3 BSS138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

Commit message: add more documentation
Other:
- net class Default removed
